File: nfdb.kicad_pcb (KiCad board)
At the start: 2 copper layers, 40 x 24 mm, 12 parts, among them J1 TYPE-C-31-M-12, J2 JST_EH_S4B-EH_1x04_P2.50mm_Ho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, J3 JST_PH_S5B-PH-K_1x05_P2.00mm_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, U1 USBLC6-2SC6

Commit message: Silk Screen Adjustment
Other:
- board text added: "Rev 1.3"
- board text removed: "Rev 1.1 RF 1"
Changed lines of the file:
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@@
     (effects (font (size 0.3 0.3) (thickness 0.06)) (justify mirror))
   )
-  (gr_text "Rev 1.1\nRF 1" (at 28.442 22.8) (layer "B.SilkS")
+  (gr_text "Rev 1.3" (at 28.442 22.8) (layer "B.SilkS")
     (effects (font (size 0.8 0.8) (thickness 0.15)) (justify mirror))
   )
